File: DRV8243 DC Motor Driver Expander/DRV8243 DC Motor Driver Expander/DRV8243 DC Motor Driver Expander.kicad_pcb (KiCad board)
At the start: 4 copper layers, 73.2 x 31.2 mm, 36 parts, among them J1 POWER, J2 CNTRL_IN, J3 CNTRL_OUT, J4 SPI, J5 MOTOR, U1 DRV8243SQRXYRQ1

Commit message: V2 Board
Parts:
- removed kibuzzard-65A7039D: G***, kibuzzard-65A7039D
- added ?: , , F.Cu at (105.7, 91.2)
- added ?: , , F.Cu at (104.3, 102.5)
- added ?: , , F.Cu at (122.5, 99.3)
- added ?: , , F.Cu at (125.7, 90.0)
- added ?: , , F.Cu at (115.9, 91.1)
- added ?: , , F.Cu at (124.2, 99.3)
- added ?: , , F.Cu at (133.3, 106.9)
- added ?: , , F.Cu at (142.2, 105.8)
- added ?: , , F.Cu at (97.7, 94.6)
- added ?: , , F.Cu at (92.6, 98.9)
- added ?: , , F.Cu at (107.4, 91.2)
- added ?: , , F.Cu at (94.4, 91.1)
- added ?: , , F.Cu at (115.9, 92.7)
- added ?: , , F.Cu at (161.2, 94.5)
- added ?: , , F.Cu at (136.3, 105.8)
- added ?: , , F.Cu at (97.7, 91.1)
- added ?: , , F.Cu at (96.1, 100.0)
- added ?: , , F.Cu at (162.7, 87.2)
- added ?: , , F.Cu at (92.6, 90.0)
- added ?: , , F.Cu at (133.3, 105.7)
- added ?: , , F.Cu at (115.9, 94.5)
- added ?: , , F.Cu at (102.4, 102.5)
- added ?: , , F.Cu at (120.9, 102.5)
- added ?: , , F.Cu at (124.2, 102.5)
- added ?: , , F.Cu at (96.0, 94.6)
- added ?: , , F.Cu at (159.8, 92.1)
- added ?: , , F.Cu at (96.0, 92.2)
- added ?: , , F.Cu at (118.0, 89.4)
- added ?: , , F.Cu at (117.4, 102.5)
- added ?: , , F.Cu at (124.2, 91.2)
- added ?: , , F.Cu at (159.7, 99.6)
- added ?: , , F.Cu at (125.8, 102.6)
- added ?: , , F.Cu at (94.5, 92.2)
- added ?: , , F.Cu at (140.7, 105.8)
- added ?: , , F.Cu at (162.8, 89.6)
- added ?: , , F.Cu at (107.6, 102.6)
- added ?: , , F.Cu at (117.9, 92.7)
- added ?: , , F.Cu at (137.8, 107.0)
- added ?: , , F.Cu at (159.7, 89.8)
- added ?: , , F.Cu at (122.3, 90.0)
- added ?: , , F.Cu at (97.4, 84.6)
- added ?: , , F.Cu at (117.5, 101.2)
- added ?: , , F.Cu at (120.8, 98.2)
- added ?: , , F.Cu at (159.7, 85.1)
- added ?: , , F.Cu at (94.4, 89.9)
- added ?: , , F.Cu at (134.8, 107.0)
- added ?: , , F.Cu at (114.2, 102.5)
- added ?: , , F.Cu at (119.0, 99.3)
- added ?: , , F.Cu at (142.2, 107.0)
- added ?: , , F.Cu at (117.9, 94.6)
- added ?: , , F.Cu at (137.8, 105.8)
- added ?: , , F.Cu at (162.8, 97.1)
- added ?: , , F.Cu at (139.2, 105.9)
- added ?: , , F.Cu at (115.9, 89.4)
- added ?: , , F.Cu at (122.5, 101.2)
- added ?: , , F.Cu at (96.0, 95.8)
- added ?: , , F.Cu at (92.7, 84.6)
- added ?: , , F.Cu at (94.5, 93.4)
- added ?: , , F.Cu at (97.7, 100.1)
- added ?: , , F.Cu at (124.1, 101.2)
- added ?: , , F.Cu at (119.0, 98.2)
- added ?: , , F.Cu at (107.4, 90.0)
- added ?: , , F.Cu at (122.5, 102.5)
- added ?: , , F.Cu at (97.4, 86.2)
- added ?: , , F.Cu at (161.2, 97.1)
- added ?: , , F.Cu at (112.3, 101.2)
- added ?: , , F.Cu at (92.7, 86.2)
- added ?: , , F.Cu at (125.8, 91.2)
- added ?: , , F.Cu at (127.1, 95.7)
- added ?: , , F.Cu at (95.0, 86.2)
- added ?: , , F.Cu at (143.7, 107.0)
- added ?: , , F.Cu at (92.6, 94.6)
- added ?: , , F.Cu at (96.0, 93.4)
- added ?: , , F.Cu at (161.2, 89.7)
- added ?: , , F.Cu at (139.2, 107.1)
- added ?: , , F.Cu at (159.8, 97.2)
- added ?: , , F.Cu at (125.8, 101.1)
- added ?: , , F.Cu at (162.8, 99.5)
- added ?: , , F.Cu at (94.5, 100.0)
- added ?: , , F.Cu at (104.1, 89.9)
- added ?: , , F.Cu at (92.6, 93.4)
- added ?: , , F.Cu at (122.3, 91.2)
- added ?: , , F.Cu at (96.0, 89.9)
- added ?: , , F.Cu at (134.8, 105.8)
- added ?: , , F.Cu at (159.7, 87.4)
- added ?: , , F.Cu at (92.6, 95.9)
- added ?: , , F.Cu at (127.1, 97.7)
- added ?: , , F.Cu at (94.5, 98.9)
- added ?: , , F.Cu at (104.1, 91.2)
- added ?: , , F.Cu at (105.9, 102.5)
- added ?: , , F.Cu at (92.8, 87.7)
- added ?: , , F.Cu at (119.0, 102.5)
- added ?: , , F.Cu at (92.6, 92.2)
- added ?: , , F.Cu at (114.2, 101.2)
- added ?: , , F.Cu at (92.6, 91.1)
- added ?: , , F.Cu at (115.8, 101.2)
- added ?: , , F.Cu at (127.0, 94.6)
- added ?: , , F.Cu at (112.3, 102.5)
- added ?: , , F.Cu at (162.8, 94.5)
- added ?: , , F.Cu at (127.4, 90.0)
- added ?: , , F.Cu at (162.9, 92.0)
- added ?: , , F.Cu at (96.0, 91.1)
- added ?: , , F.Cu at (136.3, 107.0)
- added ?: , , F.Cu at (95.1, 87.7)
- added ?: , , F.Cu at (140.7, 107.0)
- added ?: , , F.Cu at (119.0, 101.2)
- added ?: , , F.Cu at (92.6, 100.0)
- added ?: , , F.Cu at (161.2, 99.5)
- added ?: , , F.Cu at (102.2, 90.0)
- added ?: , , F.Cu at (94.4, 95.8)
- added ?: , , F.Cu at (96.1, 98.9)
- added ?: , , F.Cu at (117.9, 91.2)
- added ?: , , F.Cu at (161.3, 92.0)
- added ?: , , F.Cu at (159.8, 94.6)
- added ?: , , F.Cu at (127.1, 96.7)
- added ?: , , F.Cu at (97.7, 98.9)
- added ?: , , F.Cu at (127.5, 91.2)
- added ?: , , F.Cu at (145.3, 107.0)
- added ?: , , F.Cu at (161.1, 85.0)
- added ?: , , F.Cu at (145.3, 105.8)
- added ?: , , F.Cu at (97.7, 90.0)
- added ?: , , F.Cu at (161.1, 87.3)
- added ?: , , F.Cu at (143.7, 105.8)
- added ?: , , F.Cu at (105.7, 89.9)
- added ?: , , F.Cu at (122.5, 98.2)
- added ?: , , F.Cu at (124.1, 98.2)
- added ?: , , F.Cu at (95.0, 84.6)
- added ?: , , F.Cu at (97.5, 87.6)
- added ?: , , F.Cu at (97.8, 92.2)
- added ?: , , F.Cu at (97.8, 93.5)
- added ?: , , F.Cu at (115.8, 102.5)
- added ?: , , F.Cu at (120.8, 101.2)
- added ?: , , F.Cu at (102.3, 91.2)
- added ?: , , F.Cu at (97.7, 95.9)
- added ?: , , F.Cu at (94.4, 94.6)
- added ?: , , F.Cu at (120.9, 99.3)
- added ?: , , F.Cu at (162.7, 85.0)
- added ?: , , F.Cu at (124.1, 90.0)
- added kibuzzard-66B25C50: G***, kibuzzard-66B25C50, F.Cu at (127.3, 106.7)
- moved J5 53.4 mm to (107.5, 95.1)
- moved kibuzzard-65A6FD36 53.4 mm to (99.8, 98.6)
- moved kibuzzard-65A6FD3E 53.4 mm to (99.6, 95.0)
- moved kibuzzard-65A7001B 53.4 mm to (105.0, 96.8)
- moved G*** 46.8 mm to (151.2, 100.0)
- moved kibuzzard-65BE5B0F 30.0 mm to (112.8, 105.1)
- moved C2 21.2 mm to (138.6, 100.8), turned to 0 degrees
- moved C1 8.20 mm to (129.9, 102.3), turned to -90 degrees
- moved R1 2.46 mm to (133.7, 92.2), turned to 180 degrees
- moved C3 2.09 mm to (133.6, 89.6), turned to 180 degrees
Connections:
- U1 pad 15: (no net) -> VCC
- U1 pad 16: (no net) -> VCC
- U1 pad 17: (no net) -> VCC
- U1 pad 18: (no net) -> OUT2
- U1 pad 19: (no net) -> OUT1
- U1 pad 20: (no net) -> GND
- U1 pad 21: (no net) -> GND
Routing:
- net VCC: track 60.6 -> 16.4 mm, vias 0 -> 3
- net OUT2: track 34.1 -> 4.39 mm, vias 1 -> 3
- net OUT1: track 39.6 -> 10.4 mm, vias 1 -> 2
- net DRVOFF: track 37.4 -> 42.8 mm
- net GND: track 18.3 -> 13.9 mm, vias 10 -> 4
- net IN1: track 26.0 -> 28.2 mm
- net IN2: track 32.9 -> 34.8 mm
- net IPROPI: track 21.6 -> 19.9 mm
- net NSLEEP: track 23.8 -> 22.1 mm
- added copper zone on B.Cu, net OUT1
- added copper zone on F.Cu, net OUT1
- added copper zone on In2.Cu, net OUT1
- added copper zone on B.Cu, net OUT2
- added copper zone on F.Cu, net OUT2
- added copper zone on In2.Cu, net OUT2
- added copper zone on In2.Cu, net VCC
- removed copper zone on In2.Cu, net GND
