File: DRV8243 DC Motor Driver Expander/DRV8243 DC Motor Driver Expander/DRV8243 DC Motor Driver Expander.kicad_sch (KiCad schematic)
At the start: 14 parts, among them J1 POWER, J2 CNTRL_IN, J3 CNTRL_OUT, J4 SPI, J5 MOTOR, U1 DRV8243SQRXYRQ1

Commit message: V2 Board
Other:
- moved on the sheet: C1, C2, C3
